File: hardware/ECE477_schematic.sch (EAGLE design)
At the start: 8 parts

Commit message: adding the schematic and brd file from week 8 (midterm review)
Parts:
- removed U$1: MSP430FR69891LQFP100PIN, ECE477_parts_library:MSP430FR69891LQFP100PIN
- removed U$2: RN4020, microchip_bluetooth_v101:RN4020
- removed U$3: BUZZER, ECE477_parts_library:BUZZER
- removed U$4: CHARINGIC, ECE477_parts_library:CHARINGIC
- removed U$6: 3_3VREG, ECE477_parts_library:3_3VREG
- removed U$7: LCD, ECE477_parts_library:LCD
- removed U1: (no value), ECE477_parts_library:SIM5320
- added 2_5VREG: 2_5VREG, ECE477_parts_library:2_5VREG
- added BATTERY: JSTPH, microbuilder:JST_2PIN
- added BLUETOOTH: RN4020, microchip_bluetooth_v101:RN4020
- added BUZZER: BUZZER, ECE477_parts_library:BUZZER
- added C1, C10, C12, C13, C14, C19, C2, C20, C27, C3, C4, C5, C6, C7, C8, C9, CPUMP: (no value), rcl:C-USC1206
- added C11: 10µF, microbuilder:CAP_CERAMIC0805-NOOUTLINE
- added C15: 10pF, microbuilder:CAP_CERAMIC0805-NOOUTLINE
- added C16, C23, C24: 33pF, microbuilder:CAP_CERAMIC0805-NOOUTLINE
- added C17, C18: 100uF, rcl:C-USC1210
- added CELLMODEM: SIM5320A, ECE477_parts_library:SIM5320
- added CHARGINGIC: MCP73831T-2ACI/OT, microbuilder:MCP73831/2
- added CHRG: ORANGE, microbuilder:LED0805_NOOUTLINE
- added D1: MMSZ5231BT1G, microbuilder:DIODE-ZENERSOD123
- added DONE, NETSTATLED, POWERLED, PWRSTATLED: GREEN, microbuilder:LED0805_NOOUTLINE
- added ENABLE_SWITCH: (no value), pinhead:PINHD-1X3
- added GPSBIAS: (no value), microbuilder:SOLDERJUMPER
- added H1, H2, H3, H4: STAND-OFF, SparkFun-Hardware:STAND-OFF
- added JTAG: (no value), MSP-TS430PZ100D_v1.2:CON-ML_ML14
- added L2: 33nH, microbuilder:INDUCTOR_0805MP
- added MICROC: MSP430FR69891LQFP100PIN, ECE477_parts_library:MSP430FR69891LQFP100PIN
- added MICROUSB: MicroB, microbuilder:USBMICRO_20329
- added MOSI_TEST, SCLK_TEST: (no value), pinhead:PINHD-1X1
- added PB1, PB2, PB3: (no value), pinhead:PINHD-2X2
- added R1: 470, microbuilder:RESISTOR0805_NOOUTLINE
- added R10, R7, R8, R9: 10K, microbuilder:RESISTOR0805_NOOUTLINE
- added R2, R5, R6: 1K, microbuilder:RESISTOR0805_NOOUTLINE
- added R3: 2K, microbuilder:RESISTOR0805_NOOUTLINE
- added R4: (no value), MSP-TS430PZ100D_v1.2:SMD_R_0805
- added SMA_ANT: SMA, Adafruit FONA SIM5320 3G Breakout:MICROBUILDER_SMACONNECTOR_EDGE_UFL
- added SMF05C: SMF05C, microbuilder:TVSARRAY_5LANE
- added SW1: PANASONIC_EVQ11, MSP-TS430PZ100D_v1.2:PANASONIC_EVQ11
- added UFL: uFL, microbuilder:ANTENNA_U.FL
- added X6: SIM_LOCKAMPHENOL, microbuilder:SIM_LOCKAMPHENOL
- U$5: value 2_5VREG -> LCD; device ECE477_parts_library:2_5VREG -> ECE477_parts_library:LCD
Connections:
- new net +5V: C11.1, CHARGINGIC.VDD, CHRG.A, MICROUSB.VBUS
- new net 1.8V: CELLMODEM.V_USIM, SMF05C.C1, X6.1
- new net BLUEUART1: BLUETOOTH.5-TX, JTAG.10, MICROC.P$50
- new net BLUEUART2: BLUETOOTH.6-RX, JTAG.12, MICROC.P$51
- new net BLUEWAKEHW: BLUETOOTH.15-WAKEHW, MICROC.P$49
- new net BLUEWAKESW: BLUETOOTH.7-WAKESW, MICROC.P$48
- new net CELLRESET: CELLMODEM.RESET, MICROC.P$42
- new net CELLUART1: JTAG.14, MICROC.P$41, R5.2
- new net CELLUART2: JTAG.13, MICROC.P$40, R6.2
- new net CONNECTIONSTAT: BLUETOOTH.10-PIO1-SCK, MICROC.P$47
- new net CS: MICROC.P$5, U$5.P$18
- new net DM: CELLMODEM.USB_DM, MICROUSB.D-
- new net DP: CELLMODEM.USB_DP, MICROUSB.D+
- new net ENABLE3V3: MICROC.P$10
- new net ENABLEPB: ENABLE_SWITCH.2, MICROC.P$90
- new net GND: 2_5VREG.2, BATTERY.1, BLUETOOTH.1-GND, BLUETOOTH.24-GND, BUZZER.P$2, C1.2, C10.2, C11.2, C12.2, C13.2, C14.2, C15.2, C16.2, C17.2, C18.2, C19.2, C2.2, C20.2, C23.2, C27.2, C3.2, C4.2, C5.2, C6.2, C7.2, C8.2, C9.2, CELLMODEM.GND@1, CELLMODEM.GND@10, CELLMODEM.GND@11, CELLMODEM.GND@12, CELLMODEM.GND@13, CELLMODEM.GND@14, CELLMODEM.GND@15, CELLMODEM.GND@16, CELLMODEM.GND@17, CELLMODEM.GND@18, CELLMODEM.GND@2, CELLMODEM.GND@3, CELLMODEM.GND@4, CELLMODEM.GND@5, CELLMODEM.GND@6, CELLMODEM.GND@7, CELLMODEM.GND@8, CELLMODEM.GND@9, CHARGINGIC.VSS, D1.A, DONE.C, ENABLE_SWITCH.3, JTAG.9, MICROC.AVSS1, MICROC.AVSS2, MICROC.AVSS3, MICROC.DVSS1, MICROC.DVSS2, MICROC.DVSS3, MICROC.ESIDVSS, MICROUSB.GND, NETSTATLED.C, POWERLED.C, PWRSTATLED.C, R3.2, R7.1, R8.1, R9.1, SMA_ANT.GND1, SMA_ANT.GND2, SMA_ANT.GND3, SMA_ANT.GND4, SMF05C.A, SW1.2, U$5.P$14, U$5.P$19, UFL.GND@0, UFL.GND@1, X6.4
- new net GSM_ANT: CELLMODEM.MAIN_ANT, SMA_ANT.ANT
- new net LCDRESET: MICROC.P$3, U$5.P$20
- new net LFXIN: MICROC.P$84
- new net LFXOUT: MICROC.P$85
- new net MISO: MICROC.P$1, U$5.P$15
- new net MOSI: MICROC.P$4, MOSI_TEST.1, U$5.P$16
- new net N$1: CHRG.C, R1.1
- new net N$10: CELLMODEM.UART_TXD, R5.1
- new net N$11: CELLMODEM.UART_RXD, R6.1
- new net N$14: ENABLE_SWITCH.1, R10.1
- new net N$2: CHARGINGIC.STAT, R1.2, R2.2
- new net N$3: C20.1, U$5.P$11
- new net N$31: GPSBIAS.2, L2.1
- new net N$4: 2_5VREG.4, CPUMP.2
- new net N$5: CHARGINGIC.PROG, R3.1
- new net N$6: DONE.A, R2.1
- new net N$7: 2_5VREG.6, CPUMP.1
- new net N$8: C24.1, CELLMODEM.GPS_ANT
- new net N$9: C24.2, GPSBIAS.1, UFL.SIGNAL
- new net NETSTAT: CELLMODEM.GPIO1, NETSTATLED.A
- new net PB1: MICROC.P$94, PB1.1, R7.2
- new net PB2: MICROC.P$92, PB2.1, R8.2
- new net PB3: MICROC.P$93, PB3.1, R9.2
- new net PWM: BUZZER.P$1, MICROC.P$11
- new net PWRKEY: CELLMODEM.POWER_ON, MICROC.P$43
- new net PWRSTAT: CELLMODEM.GPIO40, PWRSTATLED.A
- new net RST: C14.1, JTAG.11, MICROC.P$29, R4.1, SW1.1
- new net SCLK: MICROC.P$2, SCLK_TEST.1, U$5.P$17
- new net SIMCLK: CELLMODEM.USIM_CLK, SMF05C.C3, X6.3
- new net SIMDATA: CELLMODEM.USIM_DATA, SMF05C.C4, X6.6
- new net SIMRST: CELLMODEM.USIM_RESET, SMF05C.C2, X6.2
- new net TCK: JTAG.7, MICROC.P$33
- new net TDI: JTAG.3, MICROC.P$31
- new net TDO: JTAG.1, MICROC.P$30
- new net TEST: JTAG.8, MICROC.P$28
- new net TMS: JTAG.5, MICROC.P$32
- new net VBAT: 2_5VREG.3, 2_5VREG.5, BATTERY.2, C13.1, C15.1, C16.1, C17.1, C18.1, C23.1, CELLMODEM.VBAT_BB@1, CELLMODEM.VBAT_BB@2, CELLMODEM.VBAT_RF@1, CELLMODEM.VBAT_RF@2, CHARGINGIC.VBAT, D1.C, L2.2, POWERLED.A
- new net VCC: 2_5VREG.1, BLUETOOTH.23-VDD, C1.1, C10.1, C12.1, C19.1, C2.1, C27.1, C3.1, C4.1, C5.1, C6.1, C7.1, C8.1, C9.1, JTAG.2, MICROC.AVCC1, MICROC.DVCC1, MICROC.DVCC2, MICROC.DVCC3, MICROC.ESIDVCC, PB1.2, PB2.2, PB3.2, R10.2, R4.2, U$5.P$12, U$5.P$13
- new net WAKEUPHOST: CELLMODEM.UART_RI, MICROC.P$39
Other:
- note added: "1.0K = 1000mA"
- note added: "10K = 100mA"
- note added: "2.0K = 500mA"
- note added: "2.5V OUT FOR VCC"
- note added: "5.0K = 200mA"
- note added: "BLUETOOTH"
- note added: "BUZZER"
- note added: "CELL MODEM"
- note added: "ESD HANDLING"
- note added: "FOR CELL MODEM"
- note added: "GSM ANTENNA"
- note added: "JTAG"
- note added: "JTAG,REST and TEST PINs"
- note added: "LCD"
- note added: "LIPO CHARGER"
- note added: "MICROCONTROLLER"
- note added: "POWER DECOUPLING"
- note added: "PUSHBUTTONS AND ENABLE SWITCH"
- note added: "SIM CARD"
- note added: "STANDOFFS"
- note added: "VCC = 2.5 V"

Commit message: the ordered PCB schematic and layout files
Parts:
- removed X6: SIM_LOCKAMPHENOL, microbuilder:SIM_LOCKAMPHENOL
- added HEARTBEAT: GREEN, microbuilder:LED0805_NOOUTLINE
- added J1: (no value), SparkFun-Connectors:SIMHOLDERSIM
- added R11: 470, microbuilder:RESISTOR0805_NOOUTLINE
- added R12, R13, R14: 1K, microbuilder:RESISTOR0805_NOOUTLINE
- C11: value 10µF -> (none); device microbuilder:CAP_CERAMIC0805-NOOUTLINE -> rcl:C-USC1206
- C15: value 10pF -> (none); device microbuilder:CAP_CERAMIC0805-NOOUTLINE -> rcl:C-USC1206
- C16, C23, C24: value 33pF -> (none); device microbuilder:CAP_CERAMIC0805-NOOUTLINE -> rcl:C-USC1206
- MICROUSB: value MicroB -> MICROB; device microbuilder:USBMICRO_20329 -> ECE477_parts_library:MICROB
- PB1, PB2, PB3: value (none) -> MOMENTARY-SWITCH-SPST-PTH-6.0MM; device pinhead:PINHD-2X2 -> SparkFun-Switches:MOMENTARY-SWITCH-SPST-PTH-6.0MM
- SMA_ANT: value SMA -> (none); device Adafruit FONA SIM5320 3G Breakout:MICROBUILDER_SMACONNECTOR_EDGE_UFL -> Adafruit FONA SIM5320 3G Breakout:MICROBUILDER_SMACONNECTOR_EDGE
- SW1: value PANASONIC_EVQ11 -> MOMENTARY-SWITCH-SPST-PTH-6.0MM; device MSP-TS430PZ100D_v1.2:PANASONIC_EVQ11 -> SparkFun-Switches:MOMENTARY-SWITCH-SPST-PTH-6.0MM
- UFL: value uFL -> (none); device microbuilder:ANTENNA_U.FL -> Adafruit FONA SIM5320 3G Breakout:MICROBUILDER_ANTENNA_U.FL
- renumbered U$5 to LCD
Connections:
- new net HEART: HEARTBEAT.A, MICROC.P$82
- new net N$12: POWERLED.C, R11.2
- new net N$13: NETSTATLED.C, R12.1
- new net N$15: PWRSTATLED.C, R13.1
- new net N$84: HEARTBEAT.C, R14.1
- net +5V: now also C11.2; no longer C11.1
- net 1.8V: now also J1.VCC; no longer X6.1
- net CS: now also MICROC.P$3; no longer MICROC.P$5
- net GND: now also C11.1, J1.GND, R11.1, R12.2, R13.2, R14.2; no longer C11.2, NETSTATLED.C, POWERLED.C, PWRSTATLED.C, X6.4
- net LCDRESET: now also MICROC.P$7; no longer MICROC.P$3
- net MISO: now also MICROC.P$5; no longer MICROC.P$1
- net PB1: now also MICROC.P$92; no longer MICROC.P$94
- net PB2: now also MICROC.P$93; no longer MICROC.P$92
- net PB3: now also MICROC.P$94; no longer MICROC.P$93
- net SIMCLK: now also J1.CLK; no longer X6.3
- net SIMDATA: now also J1.I/O; no longer X6.6
- net SIMRST: now also J1.RST; no longer X6.2
Other:
- moved on the sheet: C11, POWERLED, R9, SMA_ANT, UFL
