File: hardware/ECE477_schematic.brd (EAGLE design)
At the start: 92 x 70 mm, 67 parts, among them SW1 PANASONIC_EVQ11, X6 SIM_LOCKAMPHENOL

Commit message: the ordered PCB schematic and layout files
Parts:
- removed X6: SIM_LOCKAMPHENOL, microbuilder:C707_10M006_512_2
- added HEARTBEAT: GREEN, microbuilder:CHIPLED_0805_NOOUTLINE
- added J1: (no value), SparkFun-Connectors:SIMHOLDER
- added R11: 470, microbuilder:0805-NO
- added R12, R13, R14: 1K, microbuilder:0805-NO
- C11: value 10µF -> (none); device microbuilder:0805-NO -> rcl:C1206
- C15: value 10pF -> (none); device microbuilder:0805-NO -> rcl:C1206
- C16, C23, C24: value 33pF -> (none); device microbuilder:0805-NO -> rcl:C1206
- MICROUSB: value MicroB -> MICROB; device microbuilder:4UCONN_20329 -> ECE477_parts_library:ZX62DB5PA8(30)
- PB1, PB2, PB3: value (none) -> MOMENTARY-SWITCH-SPST-PTH-6.0MM; device pinhead:2X02 -> SparkFun-Switches:TACTILE_SWITCH_PTH_6.0MM
- SMA_ANT: value SMA -> (none); device Adafruit FONA SIM5320 3G Breakout:MICROBUILDER_SMA_EDGELAUNCH_UFL -> Adafruit FONA SIM5320 3G Breakout:MICROBUILDER_SMA_EDGELAUNCH
- SW1: value PANASONIC_EVQ11 -> MOMENTARY-SWITCH-SPST-PTH-6.0MM; device MSP-TS430PZ100D_v1.2:PANASONIC_EVQ11 -> SparkFun-Switches:TACTILE_SWITCH_PTH_6.0MM
- UFL: value uFL -> (none); device microbuilder:U.FL -> Adafruit FONA SIM5320 3G Breakout:MICROBUILDER_U.FL
- moved C24 36.7 mm to (94.1, 36.2)
- moved C15 31.9 mm to (75.2, 34.8), flipped to the bottom, turned to 0 degrees
- moved C16 30.2 mm to (76.0, 66.0), flipped to the top, turned to 0 degrees
- moved C23 26.2 mm to (89.0, 33.0)
- moved C11 7.02 mm to (79.7, 22.3), turned to 180 degrees
- moved R9 5.00 mm to (18.0, 6.00), turned to 90 degrees
- moved R8 4.12 mm to (18.0, 14.0), turned to 90 degrees
- moved R7 3.69 mm to (17.7, 21.0), turned to 90 degrees
- moved MICROUSB 3.63 mm to (96.3, 15.2)
- moved H4 3.43 mm to (96.3, 67.4)
- moved H1 3.36 mm to (96.4, 2.68)
- moved PB3 3.21 mm to (17.7, 6.19)
- moved R4 2.97 mm to (33.9, 53.7), turned to 180 degrees
- moved SW1 2.51 mm to (34.0, 54.0), turned to 0 degrees
- moved C14 2.00 mm to (31.2, 47.7)
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- renumbered U$5 to LCD
Connections:
- new net HEART: HEARTBEAT.A, MICROC.P$82
- new net N$12: POWERLED.C, R11.2
- new net N$13: NETSTATLED.C, R12.1
- new net N$15: PWRSTATLED.C, R13.1
- new net N$84: HEARTBEAT.C, R14.1
- net +5V: now also C11.2, MICROUSB.+5V; no longer C11.1, MICROUSB.VBUS
- net 1.8V: now also J1.C1; no longer X6.C1
- net CS: now also MICROC.P$3; no longer MICROC.P$5
- net GND: now also C11.1, J1.C5, R11.1, R12.2, R13.2, R14.2, SW1.3; no longer C11.2, MICROUSB.BASE@1, MICROUSB.BASE@2, MICROUSB.SPRT@1, MICROUSB.SPRT@2, MICROUSB.SPRT@3, MICROUSB.SPRT@4, NETSTATLED.C, POWERLED.C, PWRSTATLED.C, SW1.2, X6.C5
- net LCDRESET: now also MICROC.P$7; no longer MICROC.P$3
- net MISO: now also MICROC.P$5; no longer MICROC.P$1
- net PB1: now also MICROC.P$92; no longer MICROC.P$94
- net PB2: now also MICROC.P$93; no longer MICROC.P$92
- net PB3: now also MICROC.P$94; no longer MICROC.P$93
- net SIMCLK: now also J1.C3; no longer X6.C3
- net SIMDATA: now also J1.C7; no longer X6.C7
- net SIMRST: now also J1.C2; no longer X6.C2
- net VCC: now also PB1.3, PB2.3, PB3.3; no longer PB1.2, PB2.2, PB3.2
Routing:
- net GND: track 226.1 -> 68.5 mm, vias 18 -> 6
- net N$8: track 7.42 -> 43.6 mm, vias 0 -> 4
- net N$9: track 46.3 -> 11.9 mm, vias 2 -> 0
- net SIMRST: track 52.4 -> 38.6 mm
- net VBAT: track 128.2 -> 139.6 mm
- net MOSI: track 62.6 -> 74.0 mm, vias 2 -> 4
- net PB2: track 55.5 -> 44.8 mm, vias 2 -> 1
- net BLUEUART1: track 70.8 -> 81.1 mm, vias 1 -> 3
- net BLUEWAKESW: track 33.5 -> 43.3 mm
- net CELLUART2: track 35.6 -> 26.2 mm
- net PB3: track 62.0 -> 54.3 mm, vias 2 -> 1
- net VCC: track 373.8 -> 380.1 mm
- net PWM: track 40.2 -> 34.2 mm
- net N$12: track 0.00 -> 5.55 mm
- net HEART: track 0.00 -> 5.26 mm
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Other:
- board size 92 x 70 mm -> 94 x 70 mm
- board text added: "Date: 3/10/2018"
- board text added: "ECE 477 Group 16"
- board text removed: "Date: 2/27/2018"

Commit message: confirmed to be the latest
Parts:
- moved R4 0.38 mm to (33.9, 53.3), flipped to the bottom, turned to 0 degrees
Routing:
- net RST: track 51.9 -> 53.2 mm, vias 2 -> 4
Changed lines of the file:
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@@
 <attribute name="VALUE" x="88.622" y="19.502" size="0.4064" layer="27" ratio="10" rot="R90"/>
 </element>
-<element name="R4" library="MSP-TS430PZ100D_v1.2" package="SMD_0805" value="" x="33.853175" y="53.688859375" smashed="yes" rot="R180">
-<attribute name="NAME" x="34.742175" y="52.767859375" size="0.4064" layer="25" rot="R180"/>
-<attribute name="VALUE" x="34.742175" y="52.672859375" size="1.27" layer="27" rot="R180"/>
+<element name="R4" library="MSP-TS430PZ100D_v1.2" package="SMD_0805" value="" x="33.853175" y="53.311140625" smashed="yes" rot="MR0">
+<attribute name="NAME" x="34.742175" y="54.232140625" size="0.4064" layer="26" rot="MR0"/>
+<attribute name="VALUE" x="34.742175" y="54.327140625" size="1.27" layer="28" rot="MR0"/>
 </element>
 <element name="R5" library="microbuilder" package="0805-NO" value="1K" x="61.038328125" y="64.3591375" smashed="yes" rot="R180">
@@
 <wire x1="55" y1="48.6840625" x2="53.24461875" y2="46.92868125" width="0.254" layer="1"/>
 <contactref element="SW1" pad="1"/>
-<wire x1="34.792975" y1="53.688859375" x2="34.792975" y2="54.207025" width="0.8128" layer="1"/>
-<wire x1="32.7394" y1="56.2606" x2="30.7488" y2="56.2606" width="0.8128" layer="1"/>
-<wire x1="34.792975" y1="54.207025" x2="32.7394" y2="56.2606" width="0.8128" layer="1"/>
-<wire x1="29.781" y1="47.726" x2="34.792975" y2="52.737975" width="0.8128" layer="1"/>
-<wire x1="34.792975" y1="52.737975" x2="34.792975" y2="53.688859375" width="0.8128" layer="1"/>
-<wire x1="34.792975" y1="53.688859375" x2="35.104115625" y2="54" width="0.254" layer="1"/>
-<wire x1="35.104115625" y1="54" x2="39" y2="54" width="0.254" layer="1"/>
 <via x="39" y="54" extent="1-16" drill="0.35"/>
 <wire x1="41.02310625" y1="55.1377625" x2="41.4097625" y2="55.1377625" width="0.254" layer="16"/>
@@
 <wire x1="39" y1="54" x2="39.88534375" y2="54" width="0.254" layer="16"/>
 <wire x1="39.88534375" y1="54" x2="41.02310625" y2="55.1377625" width="0.254" layer="16"/>
+<wire x1="34.792975" y1="53.311140625" x2="35.311140625" y2="53.311140625" width="0.254" layer="16"/>
+<wire x1="35.311140625" y1="53.311140625" x2="36" y2="54" width="0.254" layer="16"/>
+<via x="36" y="54" extent="1-16" drill="0.35"/>
+<wire x1="36" y1="54" x2="39" y2="54" width="0.254" layer="1"/>
+<wire x1="34.792975" y1="53.311140625" x2="34.792975" y2="51.792975" width="0.8128" layer="16"/>
+<wire x1="34.792975" y1="51.792975" x2="34" y2="51" width="0.8128" layer="16"/>
+<via x="34" y="51" extent="1-16" drill="0.8"/>
+<wire x1="34" y1="51" x2="33" y2="50" width="0.8128" layer="1"/>
+<wire x1="33" y1="50" x2="31" y2="50" width="0.8128" layer="1"/>
+<wire x1="31" y1="50" x2="29.781" y2="48.781" width="0.8128" layer="1"/>
+<wire x1="29.781" y1="48.781" x2="29.781" y2="47.726" width="0.8128" layer="1"/>
+<wire x1="34.792975" y1="53.311140625" x2="34.792975" y2="54.207025" width="0.8128" layer="16"/>
+<wire x1="32.7394" y1="56.2606" x2="30.7488" y2="56.2606" width="0.8128" layer="16"/>
+<wire x1="34.792975" y1="54.207025" x2="32.7394" y2="56.2606" width="0.8128" layer="16"/>
 </signal>
 <signal name="TEST">
@@
 <wire x1="56.116515625" y1="46.605159375" x2="56.116515625" y2="44.583990625" width="0.254" layer="1"/>
 <wire x1="27" y1="53" x2="27.219134375" y2="53.219134375" width="0.8128" layer="1"/>
-<wire x1="32.913375" y1="53.688859375" x2="27.688859375" y2="53.688859375" width="0.8128" layer="1"/>
 <wire x1="41.99818125" y1="50.66518125" x2="41.99818125" y2="50.96263125" width="0.254" layer="1"/>
 <wire x1="41.99818125" y1="50.96263125" x2="41.082384375" y2="51.878428125" width="0.254" layer="1"/>
@@
 <wire x1="34.5448375" y1="46.395159375" x2="30.020934375" y2="46.395159375" width="0.254" layer="1"/>
 <via x="27.219134375" y="53.219134375" extent="1-16" drill="0.8"/>
-<wire x1="27.688859375" y1="53.688859375" x2="27.219134375" y2="53.219134375" width="0.8128" layer="1"/>
-<wire x1="27.219134375" y1="53.219134375" x2="27.25311875" y2="56.21358125" width="0.8128" layer="16"/>
+<wire x1="27.219134375" y1="53.219134375" x2="27.239315625" y2="54.997284375" width="0.8128" layer="16"/>
+<wire x1="27.239315625" y1="54.997284375" x2="27.25311875" y2="56.21358125" width="0.8128" layer="16"/>
 <wire x1="27.25311875" y1="56.21358125" x2="29" y2="58" width="0.8128" layer="16"/>
 <via x="29" y="58" extent="1-16" drill="0.8"/>
@@
 <wire x1="29.463384375" y1="65.101509375" x2="23.3106125" y2="64.937403125" width="0.8128" layer="16"/>
 <wire x1="29.463384375" y1="65.101509375" x2="27.2336125" y2="65.149403125" width="0.8128" layer="1"/>
+<wire x1="27.219134375" y1="53.219134375" x2="28" y2="54" width="0.8128" layer="16"/>
+<wire x1="32.224515625" y1="54" x2="32.913375" y2="53.311140625" width="0.8128" layer="16"/>
+<wire x1="28" y1="54" x2="32.224515625" y2="54" width="0.8128" layer="16"/>
 </signal>
 <signal name="N$12">
